File: hardware/malenki-elrs/radio.kicad_sch (KiCad schematic)
At the start: 17 parts, among them U3 SX1280IMLTRT, Y2 CRYSTAL 52MHz 10pF SMD

Commit message: Generated production files
Parts:
- C16, C19, C22: LCSC C1525 -> (none); LCSC Part # (none) -> C1525
- C18: LCSC C15195 -> (none); LCSC Part # (none) -> C15195
- C20, C29: LCSC C76988 -> (none); LCSC Part # (none) -> C76988
- C21: LCSC C47339 -> (none); LCSC Part # (none) -> C47339
- C23, C28: LCSC C76899 -> (none); LCSC Part # (none) -> C76899
- C30: LCSC C77177 -> (none); LCSC Part # (none) -> C77177
- L1: LCSC C383402 -> (none); LCSC Part # (none) -> C383402
- L2, L3: LCSC C2041661 -> (none); LCSC Part # (none) -> C2041661
- R15: LCSC C25744 -> (none); LCSC Part # (none) -> C25744
- U3: LCSC Part # (none) -> C125969
- Y2: LCSC C49253546 -> (none); LCSC Part # (none) -> C49253546; Manufacturer Seiko Epson -> (none)
Changed lines of the file:
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@@
+			)
+		)
+		(property "LCSC Part #" "C125969"
+			(at 63.5 105.41 0)
+			(hide yes)
+			(show_name no)
+			(do_not_autoplace no)
+			(effects
+				(font
+					(size 1.27 1.27)
+				)
 			)
 		)
@@
 			)
 		)
-		(property "LCSC" "C77177"
+		(property "LCSC Part #" "C77177"
 			(at 182.88 120.65 0)
 			(hide yes)
@@
 			)
 		)
-		(property "LCSC" "C1525"
+		(property "LCSC Part #" "C1525"
 			(at 111.76 66.04 0)
 			(hide yes)
@@
 			)
 		)
-		(property "LCSC" "C2041661"
+		(property "LCSC Part #" "C2041661"
 			(at 111.76 120.65 90)
 			(hide yes)
@@
 			)
 		)
-		(property "LCSC" "C1525"
+		(property "LCSC Part #" "C1525"
 			(at 78.74 66.04 0)
 			(hide yes)
@@
 			)
 		)
-		(property "LCSC" "C76899"
+		(property "LCSC Part #" "C76899"
 			(at 137.16 125.73 0)
 			(hide yes)
@@
 			)
 		)
-		(property "LCSC" "C15195"
+		(property "LCSC Part #" "C15195"
 			(at 96.52 87.63 0)
 			(hide yes)
@@
 			)
 		)
-		(property "LCSC" "C25744"
-			(at 41.91 91.44 0)
-			(hide yes)
-			(show_name no)
-			(do_not_autoplace no)
-			(effects
-				(font
-					(size 1.27 1.27)
-				)
-			)
-		)
-		(property "Manufacturer" ""
+		(property "LCSC Part #" "C25744"
 			(at 41.91 91.44 0)
 			(hide yes)
@@
 			)
 		)
-		(property "LCSC" "C76988"
+		(property "LCSC Part #" "C76988"
 			(at 146.05 110.49 0)
 			(hide yes)
@@
 			)
 		)
-		(property "LCSC" "C76988"
+		(property "LCSC Part #" "C76988"
 			(at 101.6 125.73 0)
 			(hide yes)
@@
 			)
 		)
-		(property "LCSC" "C383402"
+		(property "LCSC Part #" "C383402"
 			(at 92.71 100.33 90)
 			(hide yes)
@@
 			)
 		)
-		(property "LCSC" "C2041661"
+		(property "LCSC Part #" "C2041661"
 			(at 146.05 120.65 90)
 			(hide yes)
@@
 			)
 		)
-		(property "LCSC" "C76899"
+		(property "LCSC Part #" "C76899"
 			(at 154.94 125.73 0)
 			(hide yes)
@@
 			)
 		)
-		(property "LCSC" "C49253546"
+		(property "LCSC Part #" "C49253546"
 			(at 29.21 121.92 0)
 			(hide yes)
@@
 			)
 		)
-		(property "Manufacturer" "Seiko Epson"
-			(at 29.21 121.92 0)
-			(hide yes)
-			(show_name no)
-			(do_not_autoplace no)
-			(effects
-				(font
-					(size 1.27 1.27)
-				)
-			)
-		)
 		(pin "1"
 		)
@@
 			)
 		)
-		(property "LCSC" "C1525"
+		(property "LCSC Part #" "C1525"
 			(at 95.25 66.04 0)
 			(hide yes)
@@
 			)
 		)
-		(property "LCSC" "C47339"
+		(property "LCSC Part #" "C47339"
 			(at 102.87 101.6 0)
 			(hide yes)
